Commit message: improved dh to urdf model
- added new resources for pybullet documentation and dh to urdf paper
- implemented the new converter
- calculated joint axes and applied on robot arm ( made two versions)
- added simple constraints
- dh parameters on top of urdf file

File: outfile.urdf (robot description, URDF)
Before this commit: robot robot, 10 links, 9 joints
Links:
- added link a5; visual cylinder length=0.7 radius=0.43
- added link l5; visual cylinder length=2.0 radius=0.3
- link a0: geometry visual cylinder length=0.7 radius=0.43
- link a1: geometry visual cylinder length=0.7 radius=0.43
- link a2: geometry visual cylinder length=0.7 radius=0.43
- link a3: geometry visual cylinder length=0.7 radius=0.43
- link a4: geometry visual cylinder length=0.7 radius=0.43
- link l0: geometry visual cylinder length=2.0 radius=0.3
- link l1: geometry visual cylinder length=0.0 radius=0.3; visual cylinder length=4 radius=0.3
- link l2: geometry visual cylinder length=0.0 radius=0.3; visual cylinder length=4 radius=0.3
- link l3: geometry visual cylinder length=0.0 radius=0.3
- link l4: geometry visual cylinder length=0.0 radius=0.3
Joints:
- added joint fix_a5_to_l4: type fixed, parent l4, child a5, origin xyz=0 0 0 rpy=0 0 0
- added joint move_l5_from_a5: type revolute, parent a5, child l5, origin xyz=0.0 0.0 0.0 rpy=-1.5707963267948966 0 0, axis 0 0 1, limit lower=-2.9671 upper=2.9671 effort=12 velocity=2.6100
- joint move_l0_from_a0: axis 0.0 0.0 1.0 -> 0 0 1
- joint move_l1_from_a1: axis 0.0 0.0 1.0 -> 0 0 1; limit lower=-2.9671 upper=2.9671 effort=12 velocity=2.6100 -> lower=1 upper=4 effort=12 velocity=2.6100; origin xyz=2.0 0.0 1.0 rpy=0 0 0 -> xyz=0.0 0.0 2.0 rpy=0 0 0; type revolute -> prismatic
- joint move_l2_from_a2: axis 0.0 -1.0 6.123233995736766e-17 -> 0 0 1; limit lower=0.4 upper=4 effort=12 velocity=2.6100 -> lower=1 upper=4 effort=12 velocity=2.6100; origin xyz=2.0 0.0 1.0 rpy=0 0 0 -> xyz=0.0 0.0 0.0 rpy=-1.5707963267948966 0 0
- joint move_l3_from_a3: axis 0.0 -1.0 6.123233995736766e-17 -> 0 0 1; origin xyz=3.0 0.0 0.0 rpy=0 0 0 -> xyz=0.0 0.0 0.0 rpy=0 0 0; type fixed -> revolute
- joint move_l4_from_a4: axis 0.0 -1.0 6.123233995736766e-17 -> 0 0 1; origin xyz=2.0 0.0 2.0 rpy=0 0 0 -> xyz=0.0 0.0 0.0 rpy=1.5707963267948966 0 0

Commit message: opp for dh2urdf
- all functions done to write robot to file
- simple class to make the robot
- added utils for robotics
- added pybullet examples for robot arms
- testing serial link robot

File: outfile.urdf (robot description, URDF)
Before this commit: robot robot, 12 links, 11 joints
Links:
- removed link a4
- removed link a5
- removed link l4
- removed link l5
- link l1: geometry visual cylinder length=2.0 radius=0.3
- link l2: geometry visual cylinder length=2.0 radius=0.3; visual cylinder length=4 radius=0.3
- link l3: geometry visual cylinder length=2.0 radius=0.3
Joints:
- removed joint fix_a4_to_l3
- removed joint fix_a5_to_l4
- removed joint move_l4_from_a4
- removed joint move_l5_from_a5
- joint fix_a1_to_l0: axis (none) -> 0 0 1
- joint fix_a2_to_l1: axis (none) -> 0 0 1
- joint fix_a3_to_l2: axis (none) -> 0 0 1
- joint move_l0_from_a0: limit lower=-2.9671 upper=2.9671 effort=12 velocity=2.6100 -> lower=-3.141592653589793 upper=3.141592653589793 effort=10 velocity=2.6; origin xyz=0.0 0.0 0.0 rpy=0 0 0 -> xyz=0 0 0 rpy=0 0 0
- joint move_l1_from_a1: limit lower=1 upper=4 effort=12 velocity=2.6100 -> lower=-3.141592653589793 upper=3.141592653589793 effort=10 velocity=2.6; origin xyz=0.0 0.0 2.0 rpy=0 0 0 -> xyz=0 0 2.00000000000000 rpy=1.57079632679490 0 0; type prismatic -> revolute
- joint move_l2_from_a2: limit lower=1 upper=4 effort=12 velocity=2.6100 -> lower=0.7 upper=4 effort=10 velocity=2.6; origin xyz=0.0 0.0 0.0 rpy=-1.5707963267948966 0 0 -> xyz=2.00000000000000 0 0 rpy=1.57079632679490 0 0
- joint move_l3_from_a3: limit lower=-2.9671 upper=2.9671 effort=12 velocity=2.6100 -> lower=-3.141592653589793 upper=3.141592653589793 effort=10 velocity=2.6; origin xyz=0.0 0.0 0.0 rpy=0 0 0 -> xyz=2.00000000000000 0 0 rpy=0 0 0

Commit message: debug axes to joints
- using utils for link transform
- simple opp for serial link robot

File: outfile.urdf (robot description, URDF)
Before this commit: robot robot, 8 links, 7 joints
Links:
- removed link a3
- removed link l3
- link l1: geometry visual cylinder length=0.0 radius=0.3; visual cylinder length=4 radius=0.3
- link l2: geometry visual cylinder length=1.0 radius=0.3
Joints:
- removed joint fix_a3_to_l2
- removed joint move_l3_from_a3
- joint move_l1_from_a1: limit lower=-3.141592653589793 upper=3.141592653589793 effort=10 velocity=2.6 -> lower=0.7 upper=4 effort=10 velocity=2.6; type revolute -> prismatic
- joint move_l2_from_a2: limit lower=0.7 upper=4 effort=10 velocity=2.6 -> lower=-3.141592653589793 upper=3.141592653589793 effort=10 velocity=2.6; origin xyz=2.00000000000000 0 0 rpy=1.57079632679490 0 0 -> xyz=0 0 0 rpy=-1.57079632679490 0 0; type prismatic -> revolute
