Commit message: import existing robot arm
- importing dh param from first lines in file
- adding the constraints from the import
- class for the simulation to join multiple arms

File: my_robot.urdf (robot description, URDF)
Before this commit: robot robot, 6 links, 5 joints
Joints:
- joint move_l1_from_a1: limit lower=0.7 upper=4 effort=10 velocity=2.6 -> lower=0.8 upper=4 effort=10 velocity=2.6

Commit message: simple inverse kinematics
- using build in pybullet function for ik
- adding fixed joint to end of arm for ik
- debug text for endefector pose
- gui for ik
- updated interact

File: my_robot.urdf (robot description, URDF)
Before this commit: robot robot, 6 links, 5 joints
Links:
- added link a3; visual cylinder length=0.7 radius=0.43
- added link a4; visual cylinder length=0.7 radius=0.43
- added link a5; visual cylinder length=0.7 radius=0.43
- added link a6; visual cylinder length=0.7 radius=0.43
- added link l3; visual cylinder length=0.0 radius=0.3
- added link l4; visual cylinder length=0.0 radius=0.3
- added link l5; visual cylinder length=0.0 radius=0.3
- added link l6; visual cylinder length=0.0 radius=0.3
- link l0: geometry visual cylinder length=1.0 radius=0.3
- link l2: geometry visual cylinder length=0.0 radius=0.3; visual cylinder length=4 radius=0.3
Joints:
- added joint fix_a3_to_l2: type fixed, parent l2, child a3, origin xyz=0 0 0 rpy=0 0 0, axis 0 0 1
- added joint fix_a4_to_l3: type fixed, parent l3, child a4, origin xyz=0 0 0 rpy=0 0 0, axis 0 0 1
- added joint fix_a5_to_l4: type fixed, parent l4, child a5, origin xyz=0 0 0 rpy=0 0 0, axis 0 0 1
- added joint fix_a6_to_l5: type fixed, parent l5, child a6, origin xyz=0 0 0 rpy=0 0 0, axis 0 0 1
- added joint move_l3_from_a3: type revolute, parent a3, child l3, origin xyz=0 0 0 rpy=0 0 0, axis 0 0 1, limit lower=-3.141592653589793 upper=3.141592653589793 effort=10 velocity=2.6
- added joint move_l4_from_a4: type revolute, parent a4, child l4, origin xyz=0 0 0 rpy=1.57079632679490 0 0, axis 0 0 1, limit lower=-3.141592653589793 upper=3.141592653589793 effort=10 velocity=2.6
- added joint move_l5_from_a5: type revolute, parent a5, child l5, origin xyz=0 0 0 rpy=-1.57079632679490 0 0, axis 0 0 1, limit lower=-3.141592653589793 upper=3.141592653589793 effort=10 velocity=2.6
- added joint move_l6_from_a6: type fixed, parent a6, child l6, origin xyz=0 0 0 rpy=0 0 0, axis 0 0 1
- joint move_l1_from_a1: origin xyz=0 0 2.00000000000000 rpy=1.57079632679490 0 0 -> xyz=0 0 1.00000000000000 rpy=0 0 0
- joint move_l2_from_a2: limit lower=-3.141592653589793 upper=3.141592653589793 effort=10 velocity=2.6 -> lower=0.8 upper=4 effort=10 velocity=2.6; type revolute -> prismatic

Commit message: small fix for robot arm and dh2urdf
- save also constraints in urdf file
- cool table print for params
- improved import robot
- temporary fix for irregular movement of joints

File: my_robot.urdf (robot description, URDF)
Before this commit: robot robot, 14 links, 13 joints
Links:
- link l5: geometry visual cylinder length=2.0 radius=0.3
Joints:
- joint move_l3_from_a3: limit lower=-3.141592653589793 upper=3.141592653589793 effort=10 velocity=2.6 -> lower=-3 upper=3 effort=10 velocity=2.6
- joint move_l4_from_a4: limit lower=-3.141592653589793 upper=3.141592653589793 effort=10 velocity=2.6 -> lower=-3 upper=3 effort=10 velocity=2.6
- joint move_l5_from_a5: limit lower=-3.141592653589793 upper=3.141592653589793 effort=10 velocity=2.6 -> lower=-3 upper=3 effort=10 velocity=2.6
- joint move_l6_from_a6: origin xyz=0 0 0 rpy=0 0 0 -> xyz=2.00000000000000 0 0 rpy=0 0 0

Commit message: implemented basic trajectory functions
- move to point to simulate inverse
- move linear and circular
- write some letters and texts
- small bug at add fixed joint

File: my_robot.urdf (robot description, URDF)
Before this commit: robot robot, 14 links, 13 joints
Links:
- link l3: geometry visual cylinder length=0.1 radius=0.3
- link l4: geometry visual cylinder length=0.1 radius=0.3
Joints:
- joint move_l3_from_a3: limit lower=-3 upper=3 effort=10 velocity=2.6 -> lower=-3.141592653589793 upper=3.141592653589793 effort=10 velocity=2.6
- joint move_l4_from_a4: limit lower=-3 upper=3 effort=10 velocity=2.6 -> lower=-3.141592653589793 upper=3.141592653589793 effort=10 velocity=2.6; origin xyz=0 0 0 rpy=1.57079632679490 0 0 -> xyz=0 0 0.100000000000000 rpy=1.57079632679490 0 0
- joint move_l5_from_a5: limit lower=-3 upper=3 effort=10 velocity=2.6 -> lower=-3.141592653589793 upper=3.141592653589793 effort=10 velocity=2.6; origin xyz=0 0 0 rpy=-1.57079632679490 0 0 -> xyz=0.100000000000000 0 0 rpy=-1.57079632679490 0 0

Commit message: log robot joints
- fixed display position and orientation
- small addition to draw trajectory
- debug gui to start and stop logging
- addition to move to log immediately
- read log file
- replay gui to skim trough replay

File: my_robot.urdf (robot description, URDF)
Before this commit: robot robot, 14 links, 13 joints
Links:
- removed link a3
- removed link a4
- removed link a5
- removed link a6
- removed link l3
- removed link l4
- removed link l5
- removed link l6
- link l0: geometry visual cylinder length=3.605551275463989 radius=0.3
- link l1: geometry visual cylinder length=3.0 radius=0.3
- link l2: geometry visual cylinder length=0.0 radius=0.3
Joints:
- removed joint fix_a3_to_l2
- removed joint fix_a4_to_l3
- removed joint fix_a5_to_l4
- removed joint fix_a6_to_l5
- removed joint move_l3_from_a3
- removed joint move_l4_from_a4
- removed joint move_l5_from_a5
- removed joint move_l6_from_a6
- joint move_l1_from_a1: limit lower=0.8 upper=4 effort=10 velocity=2.6 -> lower=-2.0943951023931953 upper=2.0943951023931953 effort=10 velocity=2.6; origin xyz=0 0 1.00000000000000 rpy=0 0 0 -> xyz=3.00000000000000 0 2.00000000000000 rpy=0 0 0; type prismatic -> revolute
- joint move_l2_from_a2: limit lower=0.8 upper=4 effort=10 velocity=2.6 -> (none); origin xyz=0 0 0 rpy=-1.57079632679490 0 0 -> xyz=3.00000000000000 0 0 rpy=-1.57079632679490 0 0; type prismatic -> fixed

Commit message: adding plane point projection to move
- not can draw circles in 3d
- small fix for drawing whole circle

File: my_robot.urdf (robot description, URDF)
Before this commit: robot robot, 6 links, 5 joints
Links:
- added link a3; visual cylinder length=0.7 radius=0.43
- added link a4; visual cylinder length=0.7 radius=0.43
- added link a5; visual cylinder length=0.7 radius=0.43
- added link a6; visual cylinder length=0.7 radius=0.43
- added link l3; visual cylinder length=0.1 radius=0.3
- added link l4; visual cylinder length=0.1 radius=0.3
- added link l5; visual cylinder length=2.0 radius=0.3
- added link l6; visual cylinder length=0.0 radius=0.3
- link l0: geometry visual cylinder length=1.0 radius=0.3
- link l1: geometry visual cylinder length=0.0 radius=0.3; visual cylinder length=4 radius=0.3
- link l2: geometry visual cylinder length=0.0 radius=0.3; visual cylinder length=4 radius=0.3
Joints:
- added joint fix_a3_to_l2: type fixed, parent l2, child a3, origin xyz=0 0 0 rpy=0 0 0, axis 0 0 1
- added joint fix_a4_to_l3: type fixed, parent l3, child a4, origin xyz=0 0 0 rpy=0 0 0, axis 0 0 1
- added joint fix_a5_to_l4: type fixed, parent l4, child a5, origin xyz=0 0 0 rpy=0 0 0, axis 0 0 1
- added joint fix_a6_to_l5: type fixed, parent l5, child a6, origin xyz=0 0 0 rpy=0 0 0, axis 0 0 1
- added joint move_l3_from_a3: type revolute, parent a3, child l3, origin xyz=0 0 0 rpy=0 0 0, axis 0 0 1, limit lower=-3.141592653589793 upper=3.141592653589793 effort=10 velocity=2.6
- added joint move_l4_from_a4: type revolute, parent a4, child l4, origin xyz=0 0 0.100000000000000 rpy=1.57079632679490 0 0, axis 0 0 1, limit lower=-3.141592653589793 upper=3.141592653589793 effort=10 velocity=2.6
- added joint move_l5_from_a5: type revolute, parent a5, child l5, origin xyz=0.100000000000000 0 0 rpy=-1.57079632679490 0 0, axis 0 0 1, limit lower=-3.141592653589793 upper=3.141592653589793 effort=10 velocity=2.6
- added joint move_l6_from_a6: type fixed, parent a6, child l6, origin xyz=2.00000000000000 0 0 rpy=0 0 0, axis 0 0 1
- joint move_l1_from_a1: limit lower=-2.0943951023931953 upper=2.0943951023931953 effort=10 velocity=2.6 -> lower=0.8 upper=4 effort=10 velocity=2.6; origin xyz=3.00000000000000 0 2.00000000000000 rpy=0 0 0 -> xyz=0 0 1.00000000000000 rpy=0 0 0; type revolute -> prismatic
- joint move_l2_from_a2: limit (none) -> lower=0.8 upper=4 effort=10 velocity=2.6; origin xyz=3.00000000000000 0 0 rpy=-1.57079632679490 0 0 -> xyz=0 0 0 rpy=-1.57079632679490 0 0; type fixed -> prismatic

Commit message: include gripper
- add option to add attachments to robot
- function to control it
- simple playground to test gripper

File: my_robot.urdf (robot description, URDF)
Before this commit: robot robot, 14 links, 13 joints
Links:
- removed link a5
- removed link a6
- removed link l5
- removed link l6
- added link base, mass 1; collision cylinder length=0.15 radius=0.43; visual cylinder length=0.15 radius=0.43
- added link left_fingertip, mass 1; collision box size=0.1 .4 .1; visual mesh filename=attachments/gripper/finger.stl scale=3.7 3.7 3.7
- added link right_fingertip, mass 1; collision box size=0.1 .4 .1; visual mesh filename=attachments/gripper/finger.stl scale=3.7 3.7 3.7
- link l0: geometry visual cylinder length=3.605551275463989 radius=0.3
- link l1: geometry visual cylinder length=3.0 radius=0.3
- link l2: geometry visual cylinder length=0.0 radius=0.3; visual cylinder length=3 radius=0.3
- link l3: geometry visual cylinder length=0.0 radius=0.3
- link l4: geometry visual cylinder length=0.0 radius=0.3
Joints:
- removed joint fix_a5_to_l4
- removed joint fix_a6_to_l5
- removed joint move_l5_from_a5
- removed joint move_l6_from_a6
- added joint attachment_joint: type fixed, parent l4, child base, origin xyz=0 0 0.3 rpy=-1.5707963267948966 0 0, axis 0 0 1
- added joint base_to_left_fingertip: type prismatic, parent base, child left_fingertip, origin xyz=-0.35 -0.4 0.0, axis 1 0 0, limit lower=0 upper=0.3 effort=1.0 velocity=0.5
- added joint base_to_right_fingertip: type prismatic, parent base, child right_fingertip, origin xyz=0.35 -0.4 -0.0, axis 1 0 0, limit lower=-0.3 upper=0.0 effort=1.0 velocity=0.5
- joint move_l1_from_a1: limit lower=0.8 upper=4 effort=10 velocity=2.6 -> lower=-2.0943951023931953 upper=2.0943951023931953 effort=10 velocity=2.6; origin xyz=0 0 1.00000000000000 rpy=0 0 0 -> xyz=3.00000000000000 0 2.00000000000000 rpy=0 0 0; type prismatic -> revolute
- joint move_l2_from_a2: limit lower=0.8 upper=4 effort=10 velocity=2.6 -> lower=0.8 upper=3 effort=10 velocity=2.6; origin xyz=0 0 0 rpy=-1.57079632679490 0 0 -> xyz=3.00000000000000 0 0 rpy=-3.14159265358979 0 0
- joint move_l4_from_a4: limit lower=-3.141592653589793 upper=3.141592653589793 effort=10 velocity=2.6 -> (none); origin xyz=0 0 0.100000000000000 rpy=1.57079632679490 0 0 -> xyz=0 0 0 rpy=0 0 0; type revolute -> fixed

Commit message: add camera
- camera class to take picture
- function to find joint ids of robot
- quit simulation button
- capture image function

File: my_robot.urdf (robot description, URDF)
Before this commit: robot robot, 13 links, 12 joints
Links:
- removed link base
- removed link left_fingertip
- removed link right_fingertip
- added link a5; visual cylinder length=0.7 radius=0.43
- added link a6; visual cylinder length=0.7 radius=0.43
- added link l5; visual cylinder length=2.0 radius=0.3
- added link l6; visual cylinder length=0.0 radius=0.3
- link l0: geometry visual cylinder length=1.0 radius=0.3
- link l1: geometry visual cylinder length=0.0 radius=0.3; visual cylinder length=3 radius=0.3
- link l3: geometry visual cylinder length=0.1 radius=0.3
- link l4: geometry visual cylinder length=0.1 radius=0.3
Joints:
- removed joint attachment_joint
- removed joint base_to_left_fingertip
- removed joint base_to_right_fingertip
- added joint fix_a5_to_l4: type fixed, parent l4, child a5, origin xyz=0 0 0 rpy=0 0 0, axis 0 0 1
- added joint fix_a6_to_l5: type fixed, parent l5, child a6, origin xyz=0 0 0 rpy=0 0 0, axis 0 0 1
- added joint move_l5_from_a5: type revolute, parent a5, child l5, origin xyz=0.100000000000000 0 0 rpy=-1.57079632679490 0 0, axis 0 0 1, limit lower=-3.141592653589793 upper=3.141592653589793 effort=10 velocity=2.6
- added joint move_l6_from_a6: type fixed, parent a6, child l6, origin xyz=2.00000000000000 0 0 rpy=0 0 0, axis 0 0 1
- joint move_l1_from_a1: limit lower=-2.0943951023931953 upper=2.0943951023931953 effort=10 velocity=2.6 -> lower=0.8 upper=3 effort=10 velocity=2.6; origin xyz=3.00000000000000 0 2.00000000000000 rpy=0 0 0 -> xyz=0 0 1.00000000000000 rpy=0 0 0; type revolute -> prismatic
- joint move_l2_from_a2: origin xyz=3.00000000000000 0 0 rpy=-3.14159265358979 0 0 -> xyz=0 0 0 rpy=-1.57079632679490 0 0
- joint move_l4_from_a4: limit (none) -> lower=-3.141592653589793 upper=3.141592653589793 effort=10 velocity=2.6; origin xyz=0 0 0 rpy=0 0 0 -> xyz=0 0 0.100000000000000 rpy=1.57079632679490 0 0; type fixed -> revolute

Commit message: small fixes
- improved draw trajectory to draw multiple lines
- simple import foreign robot implementation
- moved camera and pybullet smulator to new package
- implemented new playground
- skim trough replay
- reordering of function in robot arm

File: my_robot.urdf (robot description, URDF)
Before this commit: robot robot, 14 links, 13 joints
Links:
- added link base, mass 1; collision cylinder length=0.15 radius=0.43; visual cylinder length=0.15 radius=0.43
- added link left_fingertip, mass 1; collision box size=0.1 .4 .1; visual mesh filename=attachments/gripper/finger.stl scale=3.7 3.7 3.7
- added link right_fingertip, mass 1; collision box size=0.1 .4 .1; visual mesh filename=attachments/gripper/finger.stl scale=3.7 3.7 3.7
Joints:
- added joint attachment_joint: type fixed, parent l6, child base, origin xyz=0 0 0.3 rpy=-1.5707963267948966 0 0, axis 0 0 1
- added joint base_to_left_fingertip: type prismatic, parent base, child left_fingertip, origin xyz=-0.35 -0.4 0.0, axis 1 0 0, limit lower=0 upper=0.3 effort=1.0 velocity=0.5
- added joint base_to_right_fingertip: type prismatic, parent base, child right_fingertip, origin xyz=0.35 -0.4 -0.0, axis 1 0 0, limit lower=-0.3 upper=0.0 effort=1.0 velocity=0.5
