Commit message: small fix
- find  similar log names
- fixed convert logs
- added letters
- added scaling to letters
- null space for constraints but does not work fully

File: robot_arms/mitsubishi/RV2FQ.urdf (robot description, URDF)
Before this commit: robot panda, 7 links, 6 joints
Joints:
- joint joint2: limit lower=-1.7453 upper=1.7453 effort=10 velocity=5.599666666666667 -> lower=-1.7453 upper=1.221 effort=10 velocity=5.599666666666667
- joint joint3: limit lower=0.00 upper=2.617 effort=10 velocity=6.28 -> lower=0.00 upper=2.268 effort=10 velocity=6.28

File: robot_arms/my_robot/my_robot.urdf (robot description, URDF)
Before this commit: robot robot, 13 links, 12 joints
Links:
- added link a5; visual cylinder length=0.7 radius=0.43
- added link a6; visual cylinder length=0.7 radius=0.43
- added link l5; visual cylinder length=2.0 radius=0.3
- added link l6; visual cylinder length=0.0 radius=0.3
- link l0: geometry visual cylinder length=1.0 radius=0.3
- link l1: geometry visual cylinder length=0.0 radius=0.3; visual cylinder length=3 radius=0.3
- link l3: geometry visual cylinder length=0.1 radius=0.3
- link l4: geometry visual cylinder length=0.1 radius=0.3
Joints:
- added joint fix_a5_to_l4: type fixed, parent l4, child a5, origin xyz=0 0 0 rpy=0 0 0, axis 0 0 1
- added joint fix_a6_to_l5: type fixed, parent l5, child a6, origin xyz=0 0 0 rpy=0 0 0, axis 0 0 1
- added joint move_l5_from_a5: type revolute, parent a5, child l5, origin xyz=0.100000000000000 0 0 rpy=-1.57079632679490 0 0, axis 0 0 1, limit lower=-3.141592653589793 upper=3.141592653589793 effort=10 velocity=2.6
- added joint move_l6_from_a6: type fixed, parent a6, child l6, origin xyz=2.00000000000000 0 0 rpy=0 0 0, axis 0 0 1
- joint attachment_joint: parent l4 -> l6
- joint move_l1_from_a1: limit lower=-2.0943951023931953 upper=2.0943951023931953 effort=10 velocity=2.6 -> lower=0.8 upper=3 effort=10 velocity=2.6; origin xyz=3.00000000000000 0 3.00000000000000 rpy=0 0 0 -> xyz=0 0 1.00000000000000 rpy=0 0 0; type revolute -> prismatic
- joint move_l2_from_a2: origin xyz=3.00000000000000 0 0 rpy=-3.14159265358979 0 0 -> xyz=0 0 0 rpy=-1.57079632679490 0 0
- joint move_l4_from_a4: limit (none) -> lower=-3.141592653589793 upper=3.141592653589793 effort=10 velocity=2.6; origin xyz=0 0 0 rpy=0 0 0 -> xyz=0 0 0.100000000000000 rpy=1.57079632679490 0 0; type fixed -> revolute
