Commit message: code reordering
- cleaned up init
- updated reset joints to include joint targets
- added new get robot arm joint states
- chose what to display in interact
- improved actuate attachment to change open and close targets
- move inputs all in degrees
- ik conditions for error and max frames to move
- added function to limit joints to constraints
- added new arm xarm and notebook to tinker with them

File: robot_arms/panda/panda.urdf (robot description, URDF)
Before this commit: robot panda, 13 links, 12 joints
Joints:
- removed joint panda_hand_joint
- added joint attachment_joint: type fixed, parent panda_link8, child panda_hand, origin xyz=0 0 0 rpy=0 0 -0.785398163397
