Commit message: final fixes
- capture camera orientation fixed
- added function to limit position targets
- added new revolute gripper
- added new objects to pybullet sim
- tidy up custom robot arms

File: attachments/prismatic_gripper/prismatic_gripper.urdf (robot description, URDF)
Before this commit: robot gripper, 3 links, 2 joints
Links:
- link left_fingertip: geometry collision box size=0.1 .4 .1; visual mesh filename=attachments/prismatic_gripper/finger.stl scale=3.7 3.7 3.7
- link right_fingertip: geometry collision box size=0.1 .4 .1; visual mesh filename=attachments/prismatic_gripper/finger.stl scale=3.7 3.7 3.7

File: robot_arms/mitsubishi/RV2FQ.urdf (robot description, URDF)
Before this commit: robot panda, 7 links, 6 joints
Joints:
- joint joint2: limit lower=-1.7453 upper=1.221 effort=10 velocity=5.599666666666667 -> lower=-1.7453 upper=1.7453 effort=10 velocity=5.599666666666667
- joint joint3: limit lower=0.00 upper=2.268 effort=10 velocity=6.28 -> lower=0.00 upper=2.443 effort=10 velocity=6.28

File: robot_arms/mitsubishi/RV2FQG.urdf (robot description, URDF)
Before this commit: robot panda, 10 links, 9 joints
Joints:
- joint joint2: limit lower=-1.7453 upper=1.221 effort=10 velocity=5.599666666666667 -> lower=-1.7453 upper=1.7453 effort=10 velocity=5.599666666666667
- joint joint3: limit lower=0.00 upper=2.268 effort=10 velocity=6.28 -> lower=0.00 upper=2.443 effort=10 velocity=6.28

File: robot_arms/my_robot/my_robot.urdf (robot description, URDF)
Before this commit: robot robot, 13 links, 12 joints
Links:
- removed link left_fingertip
- removed link right_fingertip
- added link left_gripper, mass 0.1; collision mesh filename=attachments/revolute_gripper/l_finger_collision.stl scale=5.7 5.7 5.7; visual mesh filename=attachments/revolute_gripper/l_finger_collision.stl scale=5.7 5.7 5.7
- added link left_tip, mass 0.1; collision mesh filename=attachments/revolute_gripper/l_finger_tip.stl scale=5.7 5.7 5.7; visual mesh filename=attachments/revolute_gripper/l_finger_tip.stl scale=5.7 5.7 5.7
- added link right_gripper, mass 0.1; collision mesh filename=attachments/revolute_gripper/l_finger_collision.stl scale=5.7 5.7 5.7; visual mesh filename=attachments/revolute_gripper/l_finger_collision.stl scale=5.7 5.7 5.7
- added link right_tip, mass 0.1; collision mesh filename=attachments/revolute_gripper/l_finger_tip.stl scale=5.7 5.7 5.7; visual mesh filename=attachments/revolute_gripper/l_finger_tip.stl scale=5.7 5.7 5.7
Joints:
- removed joint base_to_left_fingertip
- removed joint base_to_right_fingertip
- added joint left_gripper_joint: type revolute, parent base, child left_gripper, origin xyz=0.22 0.1 0 rpy=0 0 0, axis 0 0 1, limit lower=0.0 upper=0.548 effort=1000.0 velocity=0.5
- added joint left_tip_joint: type fixed, parent left_gripper, child left_tip
- added joint right_gripper_joint: type revolute, parent base, child right_gripper, origin xyz=0.22 -0.1 0 rpy=0 0 0, axis 0 0 -1, limit lower=0.0 upper=0.548 effort=1000.0 velocity=0.5
- added joint right_tip_joint: type fixed, parent right_gripper, child right_tip
- joint attachment_joint: origin xyz=0 0 0.3 rpy=-1.5707963267948966 0 0 -> xyz=0 0 0.3 rpy=0.0 -1.5707963267948966 0.0
