Commit message: mitsubishi arm
- made the custom urdf
- changed where files are saved
- load robot works with every robot
- added convert logs to prg
- break if no logs are found

File: robot_arms/my_robot/my_robot.urdf (robot description, URDF)
Before this commit: robot robot, 17 links, 16 joints
Links:
- removed link a5
- removed link a6
- removed link l5
- removed link l6
- link l0: geometry visual cylinder length=4.242640687119285 radius=0.3
- link l1: geometry visual cylinder length=3.0 radius=0.3
- link l3: geometry visual cylinder length=0.0 radius=0.3
- link l4: geometry visual cylinder length=0.0 radius=0.3
Joints:
- removed joint fix_a5_to_l4
- removed joint fix_a6_to_l5
- removed joint move_l5_from_a5
- removed joint move_l6_from_a6
- joint attachment_joint: parent l6 -> l4
- joint move_l1_from_a1: limit lower=0.8 upper=3 effort=10 velocity=2.6 -> lower=-2.0943951023931953 upper=2.0943951023931953 effort=10 velocity=2.6; origin xyz=0 0 1.00000000000000 rpy=0 0 0 -> xyz=3.00000000000000 0 3.00000000000000 rpy=0 0 0; type prismatic -> revolute
- joint move_l2_from_a2: origin xyz=0 0 0 rpy=-1.57079632679490 0 0 -> xyz=3.00000000000000 0 0 rpy=-3.14159265358979 0 0
- joint move_l4_from_a4: limit lower=-3.141592653589793 upper=3.141592653589793 effort=10 velocity=2.6 -> (none); origin xyz=0 0 0.100000000000000 rpy=1.57079632679490 0 0 -> xyz=0 0 0 rpy=0 0 0; type revolute -> fixed

Commit message: document every package
- also moved use draw and display to init
- added file name to convert to prg
- edited forces so can add an array too for every joint

File: robot_arms/my_robot/my_robot.urdf (robot description, URDF)
Before this commit: robot robot, 15 links, 14 joints
Links:
- removed link left_gripper
- removed link left_tip
- removed link right_gripper
- removed link right_tip
- added link a5; visual cylinder length=0.7 radius=0.43
- added link a6; visual cylinder length=0.7 radius=0.43
- added link l5; visual cylinder length=2.0 radius=0.3
- added link l6; visual cylinder length=0.0 radius=0.3
- added link left_fingertip, mass 1; collision box size=0.1 .4 .1; visual mesh filename=attachments/prismatic_gripper/finger.stl scale=3.7 3.7 3.7
- added link right_fingertip, mass 1; collision box size=0.1 .4 .1; visual mesh filename=attachments/prismatic_gripper/finger.stl scale=3.7 3.7 3.7
- link l0: geometry visual cylinder length=1.0 radius=0.3
- link l1: geometry visual cylinder length=0.0 radius=0.3; visual cylinder length=3 radius=0.3
- link l3: geometry visual cylinder length=0.1 radius=0.3
- link l4: geometry visual cylinder length=0.1 radius=0.3
Joints:
- removed joint left_gripper_joint
- removed joint left_tip_joint
- removed joint right_gripper_joint
- removed joint right_tip_joint
- added joint base_to_left_fingertip: type prismatic, parent base, child left_fingertip, origin xyz=-0.35 -0.4 0.0, axis 1 0 0, limit lower=0 upper=0.3 effort=1.0 velocity=0.5
- added joint base_to_right_fingertip: type prismatic, parent base, child right_fingertip, origin xyz=0.35 -0.4 -0.0, axis 1 0 0, limit lower=-0.3 upper=0.0 effort=1.0 velocity=0.5
- added joint fix_a5_to_l4: type fixed, parent l4, child a5, origin xyz=0 0 0 rpy=0 0 0, axis 0 0 1
- added joint fix_a6_to_l5: type fixed, parent l5, child a6, origin xyz=0 0 0 rpy=0 0 0, axis 0 0 1
- added joint move_l5_from_a5: type revolute, parent a5, child l5, origin xyz=0.100000000000000 0 0 rpy=-1.57079632679490 0 0, axis 0 0 1, limit lower=-3.141592653589793 upper=3.141592653589793 effort=10 velocity=2.6
- added joint move_l6_from_a6: type fixed, parent a6, child l6, origin xyz=2.00000000000000 0 0 rpy=0 0 0, axis 0 0 1
- joint attachment_joint: origin xyz=0 0 0.3 rpy=0.0 -1.5707963267948966 0.0 -> xyz=0 0 0.3 rpy=-1.5707963267948966 0.0 0.0; parent l4 -> l6
- joint move_l1_from_a1: limit lower=-2.0943951023931953 upper=2.0943951023931953 effort=10 velocity=2.6 -> lower=0.8 upper=3 effort=10 velocity=2.6; origin xyz=3.00000000000000 0 3.00000000000000 rpy=0 0 0 -> xyz=0 0 1.00000000000000 rpy=0 0 0; type revolute -> prismatic
- joint move_l2_from_a2: origin xyz=3.00000000000000 0 0 rpy=-3.14159265358979 0 0 -> xyz=0 0 0 rpy=-1.57079632679490 0 0
- joint move_l4_from_a4: limit (none) -> lower=-3.141592653589793 upper=3.141592653589793 effort=10 velocity=2.6; origin xyz=0 0 0 rpy=0 0 0 -> xyz=0 0 0.100000000000000 rpy=1.57079632679490 0 0; type fixed -> revolute

Commit message: small ease of use improvements and updated readme
- option to log the text automatically
- function to set dynamic paramteres
- improved attachment to work trough code and change the force applied when an object is detected
- first revision of docs

File: robot_arms/my_robot/my_robot.urdf (robot description, URDF)
Before this commit: robot robot, 17 links, 16 joints
Links:
- removed link a5
- removed link a6
- removed link l5
- removed link l6
- link l0: geometry visual cylinder length=4.242640687119285 radius=0.3
- link l1: geometry visual cylinder length=3.0 radius=0.3
- link l3: geometry visual cylinder length=0.0 radius=0.3
- link l4: geometry visual cylinder length=0.0 radius=0.3
Joints:
- removed joint fix_a5_to_l4
- removed joint fix_a6_to_l5
- removed joint move_l5_from_a5
- removed joint move_l6_from_a6
- joint attachment_joint: parent l6 -> l4
- joint move_l1_from_a1: limit lower=0.8 upper=3 effort=10 velocity=2.6 -> lower=-3.141592653589793 upper=3.141592653589793 effort=10 velocity=2.6; origin xyz=0 0 1.00000000000000 rpy=0 0 0 -> xyz=3.00000000000000 0 3.00000000000000 rpy=0 0 0; type prismatic -> revolute
- joint move_l2_from_a2: limit lower=0.8 upper=3 effort=10 velocity=2.6 -> lower=0.7 upper=3 effort=10 velocity=2.6; origin xyz=0 0 0 rpy=-1.57079632679490 0 0 -> xyz=3.00000000000000 0 0 rpy=-3.14159265358979 0 0
- joint move_l4_from_a4: limit lower=-3.141592653589793 upper=3.141592653589793 effort=10 velocity=2.6 -> (none); origin xyz=0 0 0.100000000000000 rpy=1.57079632679490 0 0 -> xyz=0 0 0 rpy=0 0 0; type revolute -> fixed
